File: basic-mc6800/basic-mc6800.sch (KiCad schematic (older format))
At the start: 2 parts

Commit message: Finished schmatic
Parts:
- added C? (x7): C_Small, symbol Device:C_Small
- added J?: Conn_01x39_Male, symbol Connector:Conn_01x39_Male
- added Q? (x2): Q_NMOS_DGS, symbol Device:Q_NMOS_DGS
- added R? (x2): 100k, symbol Device:R_Small
- added R? (x4): R_Small, symbol Device:R_Small
- added U?: IS61C256AL, symbol SRAM:IS61C256AL
- added U?: 74LS137, symbol 74xx:74LS137
- added Y?: 2-4Mhz, symbol Device:Crystal_GND24
Connections:
- net labels added: +5V, A0, A1, A10, A11, A12, A13, A14, A15, A2, A3, A4, A5, A6, A7, A8, A9, BA, BS, D0, D1, D2, D3, D4, D5, D6, D7, E, GND, INT1, INT2, INT3, IOREQ, M1, MEM_REQ, PER_CS, QLATCH, RESET, RO, ROM_CS, RX, R_W, TX, USR1, USR2, USR3, _A15, _QLATCH
- wire segments 0 -> 213
Other:
- note added: "0x0000-0x6FFF ROM\n0x7000 - 0x7FFF PERF\n0x8000 - 0xFFFF RAM"
- note added: "chips used:\nMC6809\n28C256\nIS61C256AL\n"
- note added: "https://www.sbprojects.net/projects/nano6802/index.php"
- note added: "when A15 high eeprom when low eeprom is active"

Commit message: mover Per_cs to pinheader
Connections:
- net labels removed: IOREQ
Other:
- note added: "0x0000 - 0x6FFF ROM\n0x7000 - 0x7FFF PERF\n0x8000 - 0xFFFF RAM"
- note added: "chips used:\nMC6809\n28C256\nIS61C256AL\n74LS137"
- note removed: "0x0000-0x6FFF ROM\n0x7000 - 0x7FFF PERF\n0x8000 - 0xFFFF RAM"
- note removed: "chips used:\nMC6809\n28C256\nIS61C256AL\n"
Changed lines of the file:
@@
 $EndComp
 Text Notes 750  1000 0    50   ~ 0
-chips used:\nMC6809\n28C256\nIS61C256AL\n
+chips used:\nMC6809\n28C256\nIS61C256AL\n74LS137
 $Comp
 L SRAM:IS61C256AL U?
@@
 Connection ~ 4350 6950
 Text Notes 1850 5200 0    50   ~ 0
-0x0000-0x6FFF ROM\n0x7000 - 0x7FFF PERF\n0x8000 - 0xFFFF RAM
+0x0000 - 0x6FFF ROM\n0x7000 - 0x7FFF PERF\n0x8000 - 0xFFFF RAM
 Text Label 2400 7050 0    50   ~ 0
 A15
@@
 Text Label 1400 5650 0    50   ~ 0
 R_W
-Text Label 1400 5850 2    50   ~ 0
-IOREQ
 Text Label 1400 5450 2    50   ~ 0
 INT1
@@
 Text Label 1400 5750 2    50   ~ 0
 RO
+Text Label 1400 5850 0    50   ~ 0
+PER_CS
 $EndSCHEMATC
