File: basic-mc6800/basic-mc6800.sch (KiCad schematic (older format))
At the start: 21 parts

Commit message: Finished routing and DRC check
Parts:
- removed Q? (x2): Q_NMOS_DGS, symbol Device:Q_NMOS_DGS
- added Q1, Q2: Q_NMOS_GSD, TO_SOT_Packages_SMD:SOT-23, symbol Device:Q_NMOS_GSD
- C1, C2, C3, C4, C5, C6, C7: renamed from C?; footprint (none) -> Capacitors_SMD:C_0603
- J1: renamed from J?; footprint (none) -> Connector_PinHeader_2.54mm:PinHeader_1x39_P2.54mm_Vertical
- R1, R2, R3, R4, R5, R6: renamed from R?; footprint (none) -> Resistor_SMD:R_0603_1608Metric
- U1: renamed from U?; footprint (none) -> Housings_SOIC:SOIC-16_3.9x9.9mm_Pitch1.27mm
- U3: renamed from U?; footprint (none) -> Housings_DIP:DIP-28_W7.62mm
- U4: renamed from U?; footprint (none) -> Housings_DIP:DIP-28_W15.24mm
- Y1: renamed from Y?; footprint (none) -> Crystal:Crystal_SMD_3225-4Pin_3.2x2.5mm
- gave numbers to parts that had none: 1
Connections:
- wire segments 213 -> 214
