File: mc6800-ioboard/mc6800-ioboard.sch (KiCad schematic (older format))
At the start: 9 parts

Commit message: schematic complete and started to route
Parts:
- added C3, C4: C_Small, Capacitor_SMD:C_0603_1608Metric, symbol Device:C_Small
- added D1, D2, D3: LED_ALT, LED_THT:LED_D5.0mm, symbol Device:LED_ALT
- added DS1: HY1602E, Display:WC1602A, symbol BAWKiCADLib:HY1602E
- added J1: Conn_01x02_Female, Connector_PinHeader_2.54mm:PinHeader_1x02_P2.54mm_Vertical, symbol Connector:Conn_01x02_Female
- added J2: Conn_01x39_Male, Connector_PinHeader_2.54mm:PinHeader_1x39_P2.54mm_Vertical, symbol Connector:Conn_01x39_Male
- added JP1: Jumper_NC_Small, Jumper:SolderJumper-2_P1.3mm_Bridged_RoundedPad1.0x1.5mm, symbol Device:Jumper_NC_Small
- added Q1: Q_NMOS_GSD, TO_SOT_Packages_SMD:SOT-23, symbol Device:Q_NMOS_GSD
- added R2, R3, R4: R_Small, Resistor_SMD:R_0603_1608Metric, symbol Device:R_Small
- added RV1: R_POT, Potentiometer_THT:Potentiometer_Vishay_T73YP_Vertical, symbol Device:R_POT
- added SW1, SW2, SW3, SW4, SW5, SW6: SW_Push, Button_Switch_SMD:SW_SPST_EVQPE1, symbol Switch:SW_Push
- added U2: 74LS32, Housings_DIP:DIP-14_W7.62mm, symbol 74xx:74LS32
- C1, C2: renamed from C?; footprint (none) -> Capacitor_SMD:C_0603_1608Metric
- R1: renamed from R?; footprint (none) -> Resistor_SMD:R_0603_1608Metric
- U1: renamed from U?; footprint (none) -> Housings_DIP:DIP-14_W7.62mm
- gave numbers to parts that had none: 1
Connections:
- net labels added: A12, A13, A14, A15, INT1, M1, MEM_RQ, RO, RX, TX, USR1, USR3
- wire segments 71 -> 198
Other:
- note added: "Address Space"
- note added: "sounder connection\n"

Commit message: more routing
Changed lines of the file:
@@
 PB.5
 Text Label 9200 5500 0    50   ~ 0
-PB.5
+PB.4
 Text Label 8500 5500 0    50   ~ 0
 PB.3

Commit message: sync checkpoint
Parts:
- added J3: USB_B, symbol Connector:USB_B
Connections:
- wire segments 198 -> 204
Changed lines of the file:
@@
 Wire Wire Line
 	1000 1400 1000 1550
+$Comp
+L Connector:USB_B J3
+U 1 1 5E683FE1
+P 4050 1150
+F 0 "J3" H 4105 1617 50  0000 C CNN
+F 1 "USB_B" H 4105 1526 50  0000 C CNN
+F 2 "" H 4200 1100 50  0001 C CNN
+F 3 " ~" H 4200 1100 50  0001 C CNN
+	1    4050 1150
+	1    0    0    -1
+$EndComp
+Wire Wire Line
+	4350 950  4850 950
+Wire Wire Line
+	4850 950  4850 800
+$Comp
+L power:+5V #PWR0121
+U 1 1 5E691506
+P 4850 800
+F 0 "#PWR0121" H 4850 650 50  0001 C CNN
+F 1 "+5V" H 4865 973 50  0000 C CNN
+F 2 "" H 4850 800 50  0001 C CNN
+F 3 "" H 4850 800 50  0001 C CNN
+	1    4850 800
+	1    0    0    -1
+$EndComp
+Wire Wire Line
+	3950 1550 3950 1700
+Wire Wire Line
+	3950 1700 4050 1700
+Wire Wire Line
+	4050 1700 4050 1550
+Wire Wire Line
+	4050 1700 4050 1900
+Connection ~ 4050 1700
+$Comp
+L power:GND #PWR0122
+U 1 1 5E6AC93F
+P 4050 1900
+F 0 "#PWR0122" H 4050 1650 50  0001 C CNN
+F 1 "GND" H 4055 1727 50  0000 C CNN
+F 2 "" H 4050 1900 50  0001 C CNN
+F 3 "" H 4050 1900 50  0001 C CNN
+	1    4050 1900
+	1    0    0    -1
+$EndComp
 $EndSCHEMATC

Commit message: checkpoint sync
Parts:
- removed DS1: HY1602E, Display:WC1602A, symbol BAWKiCADLib:HY1602E
- removed J3: USB_B, symbol Connector:USB_B
- added DS1: WC1602A, Display:WC1602A, symbol Display_Character:WC1602A
- added J3: 10118193-0001LF, digikey-footprints:USB_Micro_B_Female_10118193-0001LF, symbol dk_USB-DVI-HDMI-Connectors:10118193-0001LF
Connections:
- wire segments 204 -> 206
Changed lines of the file:
@@
 Wire Wire Line
 	2450 2600 2450 2800
-$Comp
-L BAWKiCADLib:HY1602E DS1
-U 1 1 5E640405
-P 9750 2700
-F 0 "DS1" H 9750 3678 50  0000 C CNN
-F 1 "HY1602E" H 9750 3587 50  0000 C CNN
-F 2 "Display:WC1602A" H 9750 1800 50  0001 C CIN
-F 3 "http://www.icbank.com/data/ICBShop/board/HY1602E.pdf" H 9950 2800 50  0001 C CNN
-	1    9750 2700
-	1    0    0    -1
-$EndComp
 Wire Wire Line
 	9350 2600 9000 2600
@@
 	9350 2900 9000 2900
 Wire Wire Line
-	9350 2400 9000 2400
-Wire Wire Line
 	9350 2300 9000 2300
 Wire Wire Line
+	9350 2200 9000 2200
+Wire Wire Line
 	9350 2100 9000 2100
-Wire Wire Line
-	10150 2100 10500 2100
 $Comp
 L Device:R_POT RV1
 U 1 1 5E650CF7
-P 10650 2100
-F 0 "RV1" H 10580 2054 50  0000 R CNN
-F 1 "R_POT" H 10580 2145 50  0000 R CNN
-F 2 "Potentiometer_THT:Potentiometer_Vishay_T73YP_Vertical" H 10650 2100 50  0001 C CNN
-F 3 "~" H 10650 2100 50  0001 C CNN
-	1    10650 2100
+P 10750 1600
+F 0 "RV1" H 10680 1554 50  0000 R CNN
+F 1 "R_POT" H 10680 1645 50  0000 R CNN
+F 2 "Potentiometer_THT:Potentiometer_Vishay_T73YP_Vertical" H 10750 1600 50  0001 C CNN
+F 3 "~" H 10750 1600 50  0001 C CNN
+	1    10750 1600
 	-1   0    0    1
 $EndComp
 Wire Wire Line
-	10650 2250 10650 2500
-Wire Wire Line
-	10400 2700 10400 2450
-Wire Wire Line
-	10150 2800 10400 2800
-Wire Wire Line
-	10400 2800 10400 2950
-Wire Wire Line
-	10150 2700 10400 2700
+	10750 1750 10750 2000
+Wire Wire Line
+	10400 2400 10400 2150
+Wire Wire Line
+	10150 2500 10400 2500
+Wire Wire Line
+	10400 2500 10400 2650
+Wire Wire Line
+	10150 2400 10400 2400
 Text Label 9000 2600 0    50   ~ 0
 PA.0
@@
 Text Label 9000 2100 0    50   ~ 0
 PA.4
+Text Label 9000 2200 0    50   ~ 0
+PA.5
 Text Label 9000 2300 0    50   ~ 0
-PA.5
-Text Label 9000 2400 0    50   ~ 0
 PA.6
 $Comp
@@
 L power:+5V #PWR0107
 U 1 1 5E65C89F
-P 10650 1450
-F 0 "#PWR0107" H 10650 1300 50  0001 C CNN
-F 1 "+5V" H 10665 1623 50  0000 C CNN
-F 2 "" H 10650 1450 50  0001 C CNN
-F 3 "" H 10650 1450 50  0001 C CNN
-	1    10650 1450
+P 10750 950
+F 0 "#PWR0107" H 10750 800 50  0001 C CNN
+F 1 "+5V" H 10765 1123 50  0000 C CNN
+F 2 "" H 10750 950 50  0001 C CNN
+F 3 "" H 10750 950 50  0001 C CNN
+	1    10750 950
 	1    0    0    -1
 $EndComp
@@
 L power:+5V #PWR0108
 U 1 1 5E65C8EC
-P 10400 2450
-F 0 "#PWR0108" H 10400 2300 50  0001 C CNN
-F 1 "+5V" H 10415 2623 50  0000 C CNN
-F 2 "" H 10400 2450 50  0001 C CNN
-F 3 "" H 10400 2450 50  0001 C CNN
-	1    10400 2450
+P 10400 2150
+F 0 "#PWR0108" H 10400 2000 50  0001 C CNN
+F 1 "+5V" H 10415 2323 50  0000 C CNN
+F 2 "" H 10400 2150 50  0001 C CNN
+F 3 "" H 10400 2150 50  0001 C CNN
+	1    10400 2150
 	1    0    0    -1
 $EndComp
@@
 L power:GND #PWR0111
 U 1 1 5E65C9BD
-P 10650 2500
-F 0 "#PWR0111" H 10650 2250 50  0001 C CNN
-F 1 "GND" H 10655 2327 50  0000 C CNN
-F 2 "" H 10650 2500 50  0001 C CNN
-F 3 "" H 10650 2500 50  0001 C CNN
-	1    10650 2500
+P 10750 2000
+F 0 "#PWR0111" H 10750 1750 50  0001 C CNN
+F 1 "GND" H 10755 1827 50  0000 C CNN
+F 2 "" H 10750 2000 50  0001 C CNN
+F 3 "" H 10750 2000 50  0001 C CNN
+	1    10750 2000
 	1    0    0    -1
 $EndComp
@@
 	9750 3500 9750 3850
 Wire Wire Line
-	10650 1450 10650 1950
+	10750 950  10750 1450
 Wire Wire Line
 	9750 1450 9750 1500
@@
 L power:GND #PWR0113
 U 1 1 5E668F1D
-P 10400 2950
-F 0 "#PWR0113" H 10400 2700 50  0001 C CNN
-F 1 "GND" H 10405 2777 50  0000 C CNN
-F 2 "" H 10400 2950 50  0001 C CNN
-F 3 "" H 10400 2950 50  0001 C CNN
-	1    10400 2950
+P 10400 2650
+F 0 "#PWR0113" H 10400 2400 50  0001 C CNN
+F 1 "GND" H 10405 2477 50  0000 C CNN
+F 2 "" H 10400 2650 50  0001 C CNN
+F 3 "" H 10400 2650 50  0001 C CNN
+	1    10400 2650
 	1    0    0    -1
 $EndComp
@@
 Wire Wire Line
 	1000 1400 1000 1550
-$Comp
-L Connector:USB_B J3
-U 1 1 5E683FE1
-P 4050 1150
-F 0 "J3" H 4105 1617 50  0000 C CNN
-F 1 "USB_B" H 4105 1526 50  0000 C CNN
-F 2 "" H 4200 1100 50  0001 C CNN
-F 3 " ~" H 4200 1100 50  0001 C CNN
-	1    4050 1150
-	1    0    0    -1
-$EndComp
-Wire Wire Line
-	4350 950  4850 950
-Wire Wire Line
-	4850 950  4850 800
+Wire Wire Line
+	4150 1850 4450 1850
+Wire Wire Line
+	4450 1850 4450 1700
 $Comp
 L power:+5V #PWR0121
 U 1 1 5E691506
-P 4850 800
-F 0 "#PWR0121" H 4850 650 50  0001 C CNN
-F 1 "+5V" H 4865 973 50  0000 C CNN
-F 2 "" H 4850 800 50  0001 C CNN
-F 3 "" H 4850 800 50  0001 C CNN
-	1    4850 800
-	1    0    0    -1
-$EndComp
-Wire Wire Line
-	3950 1550 3950 1700
-Wire Wire Line
-	3950 1700 4050 1700
-Wire Wire Line
-	4050 1700 4050 1550
-Wire Wire Line
-	4050 1700 4050 1900
-Connection ~ 4050 1700
+P 4450 1700
+F 0 "#PWR0121" H 4450 1550 50  0001 C CNN
+F 1 "+5V" H 4465 1873 50  0000 C CNN
+F 2 "" H 4450 1700 50  0001 C CNN
+F 3 "" H 4450 1700 50  0001 C CNN
+	1    4450 1700
+	1    0    0    -1
+$EndComp
 $Comp
 L power:GND #PWR0122
 U 1 1 5E6AC93F
-P 4050 1900
-F 0 "#PWR0122" H 4050 1650 50  0001 C CNN
-F 1 "GND" H 4055 1727 50  0000 C CNN
-F 2 "" H 4050 1900 50  0001 C CNN
-F 3 "" H 4050 1900 50  0001 C CNN
-	1    4050 1900
-	1    0    0    -1
-$EndComp
+P 4350 2850
+F 0 "#PWR0122" H 4350 2600 50  0001 C CNN
+F 1 "GND" H 4355 2677 50  0000 C CNN
+F 2 "" H 4350 2850 50  0001 C CNN
+F 3 "" H 4350 2850 50  0001 C CNN
+	1    4350 2850
+	1    0    0    -1
+$EndComp
+$Comp
+L dk_USB-DVI-HDMI-Connectors:10118193-0001LF J3
+U 1 1 5E6ACA60
+P 3850 2050
+F 0 "J3" H 3913 2795 60  0000 C CNN
+F 1 "10118193-0001LF" H 3913 2689 60  0000 C CNN
+F 2 "digikey-footprints:USB_Micro_B_Female_10118193-0001LF" H 4050 2250 60  0001 L CNN
+F 3 "http://www.amphenol-icc.com/media/wysiwyg/files/drawing/10118193.pdf" H 4050 2350 60  0001 L CNN
+F 4 "609-4616-1-ND" H 4050 2450 60  0001 L CNN "Digi-Key_PN"
+F 5 "10118193-0001LF" H 4050 2550 60  0001 L CNN "MPN"
+F 6 "Connectors, Interconnects" H 4050 2650 60  0001 L CNN "Category"
+F 7 "USB, DVI, HDMI Connectors" H 4050 2750 60  0001 L CNN "Family"
+F 8 "http://www.amphenol-icc.com/media/wysiwyg/files/drawing/10118193.pdf" H 4050 2850 60  0001 L CNN "DK_Datasheet_Link"
+F 9 "/product-detail/en/amphenol-icc-fci/10118193-0001LF/609-4616-1-ND/2785380" H 4050 2950 60  0001 L CNN "DK_Detail_Page"
+F 10 "CONN RCPT USB2.0 MICRO B SMD R/A" H 4050 3050 60  0001 L CNN "Description"
+F 11 "Amphenol ICC (FCI)" H 4050 3150 60  0001 L CNN "Manufacturer"
+F 12 "Active" H 4050 3250 60  0001 L CNN "Status"
+	1    3850 2050
+	1    0    0    -1
+$EndComp
+Wire Wire Line
+	4150 2250 4350 2250
+Wire Wire Line
+	4350 2250 4350 2800
+Wire Wire Line
+	3750 2650 3750 2800
+Wire Wire Line
+	3750 2800 4350 2800
+Connection ~ 4350 2800
+Wire Wire Line
+	4350 2800 4350 2850
+$Comp
+L Display_Character:WC1602A DS1
+U 1 1 5E72943A
+P 9750 2700
+F 0 "DS1" H 9750 3678 50  0000 C CNN
+F 1 "WC1602A" H 9750 3587 50  0000 C CNN
+F 2 "Display:WC1602A" H 9750 1800 50  0001 C CIN
+F 3 "http://www.wincomlcd.com/pdf/WC1602A-SFYLYHTC06.pdf" H 10450 2700 50  0001 C CNN
+	1    9750 2700
+	1    0    0    -1
+$EndComp
+Wire Wire Line
+	10150 2100 10150 1600
+Wire Wire Line
+	10150 1600 10600 1600
 $EndSCHEMATC
